Commit message: Final Changes

File: body.urdf (robot description, URDF)
Before this commit: robot robot, 3 links, 2 joints
Links:
- added link Backfoot, mass 1; collision box size=0.2 0.2 1; visual box size=0.2 0.2 1
- added link Frontfoot, mass 1; collision box size=0.2 0.2 1; visual box size=0.2 0.2 1
- added link Leftfoot, mass 1; collision box size=0.2 0.2 1; visual box size=0.2 0.2 1
- added link Leftleg, mass 1; collision box size=1 0.2 0.2; visual box size=1 0.2 0.2
- added link Rightfoot, mass 1; collision box size=0.2 0.2 1; visual box size=0.2 0.2 1
- added link Rightleg, mass 1; collision box size=1 0.2 0.2; visual box size=1 0.2 0.2
- link Backleg: geometry collision box size=0.2 1 0.2; visual box size=0.2 1 0.2
- link Frontleg: geometry collision box size=0.2 1 0.2; visual box size=0.2 1 0.2
Joints:
- added joint Backleg_Backfoot: type revolute, parent Backleg, child Backfoot, origin xyz=0 -1 0 rpy=0 0 0, axis 1 0 0, limit lower=-3.14159 upper=3.14159 effort=0.0 velocity=0.0
- added joint Frontleg_Frontfoot: type revolute, parent Frontleg, child Frontfoot, origin xyz=0 1 0 rpy=0 0 0, axis 1 0 0, limit lower=-3.14159 upper=3.14159 effort=0.0 velocity=0.0
- added joint Leftleg_Leftfoot: type revolute, parent Leftleg, child Leftfoot, origin xyz=-1 0 0 rpy=0 0 0, axis 0 1 0, limit lower=-3.14159 upper=3.14159 effort=0.0 velocity=0.0
- added joint Rightleg_Rightfoot: type revolute, parent Rightleg, child Rightfoot, origin xyz=1 0 0 rpy=0 0 0, axis 0 1 0, limit lower=-3.14159 upper=3.14159 effort=0.0 velocity=0.0
- added joint Torso_Leftleg: type revolute, parent Torso, child Leftleg, origin xyz=-0.5 0 1 rpy=0 0 0, axis 0 1 0, limit lower=-3.14159 upper=3.14159 effort=0.0 velocity=0.0
- added joint Torso_Rightleg: type revolute, parent Torso, child Rightleg, origin xyz=0.5 0 1 rpy=0 0 0, axis 0 1 0, limit lower=-3.14159 upper=3.14159 effort=0.0 velocity=0.0
- joint Torso_Backleg: axis 0 1 0 -> 1 0 0; origin xyz=0.5 0 1 rpy=0 0 0 -> xyz=0 -0.5 1 rpy=0 0 0
- joint Torso_Frontleg: axis 0 1 0 -> 1 0 0; origin xyz=-0.5 0 1 rpy=0 0 0 -> xyz=0 0.5 1 rpy=0 0 0

Commit message: It Topples Like a Tree

File: body.urdf (robot description, URDF)
Before this commit: robot robot, 9 links, 8 joints
Links:
- removed link Backfoot
- removed link Backleg
- removed link Frontfoot
- removed link Frontleg
- added link Leftarm, mass 1; collision box size=0.2 0.2 1; visual box size=0.2 0.2 1
- added link Lefthand, mass 1; collision box size=0.2 0.2 1; visual box size=0.2 0.2 1
- added link Leftshin, mass 1; collision box size=0.2 0.2 2; visual box size=0.2 0.2 2
- added link Rightarm, mass 1; collision box size=0.2 0.2 1; visual box size=0.2 0.2 1
- added link Righthand, mass 1; collision box size=0.2 0.2 1; visual box size=0.2 0.2 1
- added link Rightshin, mass 1; collision box size=0.2 0.2 2; visual box size=0.2 0.2 2
- link Leftfoot: geometry collision box size=1 0.2 0.2; visual box size=1 0.2 0.2
- link Leftleg: geometry collision box size=0.2 0.2 2; visual box size=0.2 0.2 2
- link Rightfoot: geometry collision box size=1 0.2 0.2; visual box size=1 0.2 0.2
- link Rightleg: geometry collision box size=0.2 0.2 2; visual box size=0.2 0.2 2
- link Torso: geometry collision box size=0.5 1 2; visual box size=0.5 1 2
Joints:
- removed joint Backleg_Backfoot
- removed joint Frontleg_Frontfoot
- removed joint Leftleg_Leftfoot
- removed joint Rightleg_Rightfoot
- removed joint Torso_Backleg
- removed joint Torso_Frontleg
- added joint Leftarm_Lefthand: type revolute, parent Leftarm, child Lefthand, origin xyz=0 0 -1 rpy=0 0 0, axis 0 1 0, limit lower=-3.14159 upper=3.14159 effort=0.0 velocity=0.0
- added joint Leftleg_Leftshin: type revolute, parent Leftleg, child Leftshin, origin xyz=0 0 -2 rpy=0 0 0, axis 0 1 0, limit lower=-3.14159 upper=3.14159 effort=0.0 velocity=0.0
- added joint Leftshin_Leftfoot: type revolute, parent Leftshin, child Leftfoot, origin xyz=0 0 -2 rpy=0 0 0, axis 0 1 0, limit lower=-3.14159 upper=3.14159 effort=0.0 velocity=0.0
- added joint Rightarm_Righthand: type revolute, parent Rightarm, child Righthand, origin xyz=0 0 -1 rpy=0 0 0, axis 0 1 0, limit lower=-3.14159 upper=3.14159 effort=0.0 velocity=0.0
- added joint Rightleg_Rightshin: type revolute, parent Rightleg, child Rightshin, origin xyz=0 0 -2 rpy=0 0 0, axis 0 1 0, limit lower=-3.14159 upper=3.14159 effort=0.0 velocity=0.0
- added joint Rightshin_Rightfoot: type revolute, parent Rightshin, child Rightfoot, origin xyz=0 0 -2 rpy=0 0 0, axis 0 1 0, limit lower=-3.14159 upper=3.14159 effort=0.0 velocity=0.0
- added joint Torso_Leftarm: type revolute, parent Torso, child Leftarm, origin xyz=0 -0.6 5.7 rpy=0 0 0, axis 0 1 0, limit lower=-3.14159 upper=3.14159 effort=0.0 velocity=0.0
- added joint Torso_Rightarm: type revolute, parent Torso, child Rightarm, origin xyz=0 0.6 5.7 rpy=0 0 0, axis 0 1 0, limit lower=-3.14159 upper=3.14159 effort=0.0 velocity=0.0
- joint Torso_Leftleg: origin xyz=-0.5 0 1 rpy=0 0 0 -> xyz=0 -0.25 4.2 rpy=0 0 0
- joint Torso_Rightleg: origin xyz=0.5 0 1 rpy=0 0 0 -> xyz=0 0.25 4.2 rpy=0 0 0
